File: PCBModel/GoBabyGo.kicad_sch (KiCad schematic)
At the start: 27 parts, among them J1 Conn_01x02_Pin, Q1 Q_NPN_BCE, Q2 Q_NPN_BCE, U1 NE555P, U2 NE555P

Commit message: PCB review.
Parts:
- removed Q1, Q2: Q_NPN_BCE, Package_TO_SOT_THT:TO-92_Wide, symbol Transistor_BJT:Q_NPN_BCE
- added JP5: Jumper_GND, Resistor_THT:R_Axial_DIN0207_L6.3mm_D2.5mm_P5.08mm_Vertical, symbol Jumper:Jumper_2_Bridged
- added Q1, Q2: NPN, Package_TO_SOT_THT:TO-92_Wide, symbol Simulation_SPICE:NPN
Connections:
- net GND: now also JP5.1 (A), JP5.2 (B), Q1.3 (E), Q2.3 (E)
- net at R12.2: now also Q1.2 (B)
- net at R14.1, U2.2 (TRIG): now also Q1.1 (C)
- net at R3.2: now also Q2.2 (B)
- net at R4.1, U1.2 (TRIG): now also Q2.1 (C)
Other:
- moved on the sheet: J1, JP1, JP2, JP3, JP4

Commit message: schematic update
Parts:
- added M1, M2, M3, M4: Motor_DC, symbol Motor:Motor_DC
- added U3: R-78E5.0-0.5, Converter_DCDC:Converter_DCDC_RECOM_R-78E-0.5_THT, symbol Converter_DCDC:R-78E5.0-0.5
Connections:
- net +5V: now also U3.3 (OUT)
- net GND: now also U3.2 (GND)
- new net +12V: U3.1 (IN)

Commit message: Start of the README Report
Parts:
- removed M3, M4: Motor_DC, symbol Motor:Motor_DC
Connections:
- net +12V: now also M1.1 (+), M2.1 (+)
- net GND: now also M1.2 (-), M2.2 (-)
Other:
- moved on the sheet: M1, M2
